Commit message: Add collision shapes and repair links

File: models/onrobot_sg_b/sg_b.urdf (robot description, URDF)
Before this commit: robot sg-b, 2 links, 1 joints
Links:
- link gripper: geometry collision cylinder length=0.115 radius=0.049; visual mesh filename=package://onrobot_sg/models/onrobot_sg_b/meshes/SG-b_v1.dae scale=1 1 1
- link quick_change_robot_side: geometry collision cylinder length=0.015 radius=0.036; visual mesh filename=package://onrobot_sg/models/common/Quick_Changer_Robot Side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 scale=1 1 1
Joints:
- joint quick_changer_to_gripper: origin xyz=-0.0055 -.024 0.0075 rpy=0 0 -1.5708 -> xyz=0 0 0.024 rpy=0 0 0
